File: RP2040_Injector.kicad_sch (KiCad schematic)
At the start: 25 parts, among them J1 USB-A, J2 Conn_01x02, U1 NCP1117-3.3_SOT223, U2 W25Q128JVS, U3 RP2040

Commit message: Finalized v0.1 design
Parts:
- added D1: LED, LED_SMD:LED_0603_1608Metric, symbol Device:LED
- added R1: 2k2, Resistor_SMD:R_0402_1005Metric, symbol Device:R
- renumbered R1 to R2, R2 to R3, R3 to R4
Connections:
- net +3V3: now also D1.2 (A)
- net GND: now also R1.2
- new net: D1.1 (K), R1.1
Changed lines of the file:
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@@
   (junction (at 225.425 41.91) (diameter 0) (color 0 0 0 0)
   )
+  (junction (at 95.25 41.91) (diameter 0) (color 0 0 0 0)
+  )
   (junction (at 137.16 31.115) (diameter 0) (color 0 0 0 0)
+  )
+  (junction (at 99.06 31.115) (diameter 0) (color 0 0 0 0)
   )
   (junction (at 95.25 31.115) (diameter 0) (color 0 0 0 0)
@@
     (stroke (width 0) (type default) (color 0 0 0 0))
   )
+  (wire (pts (xy 111.125 41.91) (xy 95.25 41.91))
+    (stroke (width 0) (type default) (color 0 0 0 0))
+  )
   (wire (pts (xy 163.83 40.005) (xy 163.83 41.91))
     (stroke (width 0) (type default) (color 0 0 0 0))
@@
     (stroke (width 0) (type default) (color 0 0 0 0))
   )
+  (wire (pts (xy 99.06 31.115) (xy 103.505 31.115))
+    (stroke (width 0) (type default) (color 0 0 0 0))
+  )
   (wire (pts (xy 133.35 44.45) (xy 133.35 41.91))
     (stroke (width 0) (type default) (color 0 0 0 0))
@@
     (stroke (width 0) (type default) (color 0 0 0 0))
   )
+  (wire (pts (xy 111.125 31.115) (xy 111.125 33.02))
+    (stroke (width 0) (type default) (color 0 0 0 0))
+  )
   (wire (pts (xy 223.52 76.2) (xy 223.52 95.25))
     (stroke (width 0) (type default) (color 0 0 0 0))
@@
   )
   (wire (pts (xy 83.82 93.345) (xy 83.82 97.155))
+    (stroke (width 0) (type default) (color 0 0 0 0))
+  )
+  (wire (pts (xy 111.125 40.64) (xy 111.125 41.91))
     (stroke (width 0) (type default) (color 0 0 0 0))
   )
@@
   (symbol (lib_id "power:+1V1") (at 212.725 28.575 0) (unit 1)
     (in_bom yes) (on_board yes)
-    (property "Reference" "#PWR?" (id 0) (at 212.725 32.385 0)
+    (property "Reference" "#PWR05" (id 0) (at 212.725 32.385 0)
       (effects (font (size 1.27 1.27)) hide)
     )
@@
   (symbol (lib_id "Device:R") (at 137.16 99.695 90) (unit 1)
     (in_bom yes) (on_board yes)
-    (property "Reference" "R1" (id 0) (at 137.16 95.885 90))
+    (property "Reference" "R2" (id 0) (at 137.16 95.885 90))
     (property "Value" "1k" (id 1) (at 137.16 97.79 90))
     (property "Footprint" "Resistor_SMD:R_0402_1005Metric" (id 2) (at 137.16 101.473 90)
@@
   (symbol (lib_id "Device:R") (at 92.71 130.81 270) (unit 1)
     (in_bom yes) (on_board yes)
-    (property "Reference" "R2" (id 0) (at 92.71 128.905 90))
+    (property "Reference" "R3" (id 0) (at 92.71 128.905 90))
     (property "Value" "27" (id 1) (at 92.71 130.81 90))
     (property "Footprint" "Resistor_SMD:R_0402_1005Metric" (id 2) (at 92.71 129.032 90)
@@
   (symbol (lib_id "Device:R") (at 92.71 137.16 270) (unit 1)
     (in_bom yes) (on_board yes)
-    (property "Reference" "R3" (id 0) (at 92.71 135.255 90))
+    (property "Reference" "R4" (id 0) (at 92.71 135.255 90))
     (property "Value" "27" (id 1) (at 92.71 137.16 90))
     (property "Footprint" "Resistor_SMD:R_0402_1005Metric" (id 2) (at 92.71 135.382 90)
@@
     )
     (property "Datasheet" "~" (id 3) (at 216.535 36.195 0)
+      (effects (font (size 1.27 1.27)) hide)
+    )
+    (pin "1")
+    (pin "2")
+  )
+  (symbol (lib_id "Device:LED") (at 107.315 31.115 180) (unit 1)
+    (in_bom yes) (on_board yes) (fields_autoplaced)
+    (property "Reference" "D1" (id 0) (at 108.9025 24.13 0))
+    (property "Value" "LED" (id 1) (at 108.9025 26.67 0))
+    (property "Footprint" "LED_SMD:LED_0603_1608Metric" (id 2) (at 107.315 31.115 0)
+      (effects (font (size 1.27 1.27)) hide)
+    )
+    (property "Datasheet" "~" (id 3) (at 107.315 31.115 0)
       (effects (font (size 1.27 1.27)) hide)
     )
@@
     (pin "2")
   )
+  (symbol (lib_id "Device:R") (at 111.125 36.83 0) (unit 1)
+    (in_bom yes) (on_board yes) (fields_autoplaced)
+    (property "Reference" "R1" (id 0) (at 113.03 35.5599 0)
+      (effects (font (size 1.27 1.27)) (justify left))
+    )
+    (property "Value" "2k2" (id 1) (at 113.03 38.0999 0)
+      (effects (font (size 1.27 1.27)) (justify left))
+    )
+    (property "Footprint" "Resistor_SMD:R_0402_1005Metric" (id 2) (at 109.347 36.83 90)
+      (effects (font (size 1.27 1.27)) hide)
+    )
+    (property "Datasheet" "~" (id 3) (at 111.125 36.83 0)
+      (effects (font (size 1.27 1.27)) hide)
+    )
+    (pin "1")
+    (pin "2")
+  )
   (symbol (lib_id "power:+3V3") (at 34.29 109.855 90) (unit 1)
     (in_bom yes) (on_board yes)
@@
       (reference "#PWR04") (unit 1) (value "+3V3") (footprint "")
     )
+    (path "/0242ac6c-6f75-41c5-a366-4aa2f3994564"
+      (reference "#PWR05") (unit 1) (value "+1V1") (footprint "")
+    )
     (path "/ec98bcfc-0663-40ee-b1b9-ced19fbe610c"
       (reference "#PWR06") (unit 1) (value "GND") (footprint "")
@@
       (reference "#PWR018") (unit 1) (value "GND") (footprint "")
     )
-    (path "/0242ac6c-6f75-41c5-a366-4aa2f3994564"
-      (reference "#PWR?") (unit 1) (value "+1V1") (footprint "")
-    )
     (path "/642caec6-d059-45a8-9333-e52015b8e2b0"
       (reference "C1") (unit 1) (value "10u") (footprint "Capacitor_SMD:C_0805_2012Metric")
@@
       (reference "C16") (unit 1) (value "15p") (footprint "Capacitor_SMD:C_0402_1005Metric")
     )
+    (path "/b73c6e7c-769a-4761-b90d-a74ffcc4eb71"
+      (reference "D1") (unit 1) (value "LED") (footprint "LED_SMD:LED_0603_1608Metric")
+    )
     (path "/fc5802ea-4034-45a1-97e1-ef224a2e8b27"
       (reference "HSE1") (unit 1) (value "12MHz") (footprint "Crystal:Crystal_SMD_SeikoEpson_FA238-4Pin_3.2x2.5mm")
@@
       (reference "J2") (unit 1) (value "Conn_01x02") (footprint "Connector_PinHeader_2.54mm:PinHeader_1x02_P2.54mm_Vertical")
     )
+    (path "/c511aec4-e6a0-465c-abdc-1868336933d1"
+      (reference "R1") (unit 1) (value "2k2") (footprint "Resistor_SMD:R_0402_1005Metric")
+    )
     (path "/7c963190-4511-4c0e-8902-b004f52d4d25"
-      (reference "R1") (unit 1) (value "1k") (footprint "Resistor_SMD:R_0402_1005Metric")
+      (reference "R2") (unit 1) (value "1k") (footprint "Resistor_SMD:R_0402_1005Metric")
     )
     (path "/7dd2e861-7829-452d-bfa5-328e9ca8343b"
-      (reference "R2") (unit 1) (value "27") (footprint "Resistor_SMD:R_0402_1005Metric")
+      (reference "R3") (unit 1) (value "27") (footprint "Resistor_SMD:R_0402_1005Metric")
     )
     (path "/7e2e4fd2-38ff-43af-b4a8-a0f5a20d3e88"
-      (reference "R3") (unit 1) (value "27") (footprint "Resistor_SMD:R_0402_1005Metric")
+      (reference "R4") (unit 1) (value "27") (footprint "Resistor_SMD:R_0402_1005Metric")
     )
     (path "/03e319ea-83a0-43a9-b383-949ba2b66eab"

Commit message: Started v0.2
Parts:
- added F1: 0805L050WR, Fuse:Fuse_0805_2012Metric, symbol Device:Polyfuse
- added R2: 1k, Resistor_SMD:R_0402_1005Metric, symbol Device:R
- C14: renamed from C15; value 15p -> 20p
- C15: renamed from C16; value 15p -> 20p
- J2: footprint Connector_PinHeader_2.54mm:PinHeader_1x02_P2.54mm_Vertical -> Connector_PinHeader_2.00mm:PinHeader_1x02_P2.00mm_Vertical
- renumbered C3 to C1, C12 to C10, C13 to C11, C1 to C12, C2 to C13, C14 to C16, C4 to C2, C5 to C3, C6 to C4, C7 to C5, C8 to C6, C9 to C7, C10 to C8, C11 to C9, R2 to R5, U3 to U2, U2 to U3
Connections:
- net VCC: now also F1.1; no longer C12.1, U1.3 (VI)
- net XOUT: now also R2.2; no longer C15.1, HSE1.3
- net USB_DM renamed USB_D-
- net USB_DP renamed USB_D+
- new net: C12.1, F1.2, U1.3 (VI)
- new net: C15.1, HSE1.3, R2.1
Other:
- moved on the sheet: C1, C10, C11, C12, C13, C14, C15, C16, C2, C3, C4, C5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
